File: resources/KiCad/04_GoBananas/04_GoBananas.kicad_sch (KiCad schematic)
At the start: 3 parts

Commit message: 04_GoBananas schematic
Parts:
- added LS1: Speaker, symbol Device:Speaker
Connections:
- net at A?.~ (VIN): now also A1.~ (USB-_15)
- net at R1.1: now also A1.~ (USB-_15); no longer A?.~ (VIN)
- net at A1.~ (USB-_15): no longer A?.~ (VIN)
- net at R1.2: now also A?.~ (VIN); no longer A1.~ (USB-_15)
- new net: A1.~ (USB-_15), A?.~ (VIN) (x3)
- new net: A1.~ (USB-_15), LS1.1
- new net: A1.~ (USB-_15), LS1.2
- now unconnected: A1.~ (USB-_15), A1.~ (USB-_15), A1.~ (USB-_15)
Other:
- note added: "Connections to Sound Circuitry: (YX5200/DFPlayer) | YX5200 | Color | Arduino | | --- | --- | --- | | 03_TX | Blue | 02 | | 02_RX | Green | 03 resistor | | Busy_16 | Yellow | 04 | | PWR | Red | 5V | | GND | Black | GND |"
- note added: "Red"
- note removed: "Connections to Sound Circuitry: (YX5200/DFPlayer) | YX5200 | Color | Arduino | | --- | --- | --- | | 03_TX | Blue | 02 | | 02_RX | Green | 03 | | Busy_16 | Yellow | 04 | | PWR | Red | 5V | | GND | Black | GND |"
- moved on the sheet: A1A, R1
