File: resources/KiCad/03_BigSonarProject/03_BigSonarProject.kicad_sch (KiCad schematic)
At the start: 6 parts

Commit message: some updates for 03
Connections:
- net at A?.~ (VIN), M?.~ (VCC): now also Z?.~ (GND); no longer SW?.2
- net at Z?.~ (GND): no longer A?.~ (VIN)
- new net: A?.~ (VIN), SW?.2
- new net: A?.~ (VIN), M?.~ (VCC) (x3)
Other:
- note added: "Battery"
- note added: "Switch is unused"
- note removed: "9V Battery"
Changed lines of the file:
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@@
   (title_block
     (title "03 Big Sonar Range Detector")
-    (date "2024-05-01")
+    (date "2024-06-14")
     (company "Author: https://github.com/Mark-MDO47")
     (comment 1 "NOTE: Chips & Modules shown top view, notch at top")
@@
   (junction (at 90.17 83.82) (diameter 0) (color 0 0 0 0)
   )
-  (junction (at 137.16 123.19) (diameter 0) (color 0 0 0 0)
+  (junction (at 182.88 118.11) (diameter 0) (color 0 0 0 0)
   )
   (junction (at 90.17 93.98) (diameter 0) (color 0 0 0 0)
@@
     (stroke (width 0) (type default))
   )
-  (wire (pts (xy 115.57 146.05) (xy 111.76 146.05))
+  (wire (pts (xy 100.33 96.52) (xy 123.19 96.52))
     (stroke (width 0) (type default))
   )
-  (wire (pts (xy 100.33 104.14) (xy 100.33 114.3))
+  (wire (pts (xy 100.33 96.52) (xy 100.33 114.3))
     (stroke (width 0) (type default))
   )
@@
     (stroke (width 0) (type default))
   )
-  (wire (pts (xy 137.16 123.19) (xy 137.16 142.24))
-    (stroke (width 0) (type default))
-  )
-  (wire (pts (xy 100.33 104.14) (xy 123.19 104.14))
-    (stroke (width 0) (type default))
-  )
   (wire (pts (xy 179.07 123.19) (xy 179.07 166.37))
     (stroke (width 0) (type default))
@@
     (stroke (width 0) (type default))
   )
-  (wire (pts (xy 123.19 81.28) (xy 123.19 104.14))
+  (wire (pts (xy 123.19 81.28) (xy 123.19 96.52))
     (stroke (width 0) (type default))
   )
@@
     (stroke (width 0) (type default))
   )
-  (wire (pts (xy 115.57 142.24) (xy 115.57 146.05))
+  (wire (pts (xy 111.76 146.05) (xy 120.65 146.05))
+    (stroke (width 0) (type default))
+  )
+  (wire (pts (xy 120.65 105.41) (xy 182.88 105.41))
     (stroke (width 0) (type default))
   )
@@
   )
   (wire (pts (xy 143.51 128.27) (xy 123.19 128.27))
+    (stroke (width 0) (type default))
+  )
+  (wire (pts (xy 120.65 105.41) (xy 120.65 146.05))
     (stroke (width 0) (type default))
   )
@@
   )
   (wire (pts (xy 50.8 85.09) (xy 50.8 83.82))
-    (stroke (width 0) (type default))
-  )
-  (wire (pts (xy 137.16 142.24) (xy 115.57 142.24))
     (stroke (width 0) (type default))
   )
@@
     (stroke (width 0) (type default))
   )
-  (text "Resistor is optional" (at 101.6 111.76 0)
+  (wire (pts (xy 182.88 105.41) (xy 182.88 118.11))
+    (stroke (width 0) (type default))
+  )
+  (text "Resistor is optional" (at 68.58 118.11 0)
     (effects (font (size 2 2)) (justify left bottom))
   )
-  (text "9V Battery" (at 48.26 81.28 0)
+  (text "Battery" (at 48.26 81.28 0)
     (effects (font (size 1.27 1.27)) (justify left bottom))
   )
+  (text "Switch is unused" (at 121.92 113.03 0)
+    (effects (font (size 2 2)) (justify left bottom))
+  )
   (symbol (lib_id "Device:R_Small_US") (at 100.33 116.84 0) (unit 1)

Commit message: update PDF
Parts:
- added SW1: SW_SPST, symbol MDO:SW_SPST
Connections:
- net at A?.~ (VIN): now also M?.~ (VCC), Z?.~ (GND)
- net at BT?.1 (+): now also SW1.~ (B)
- new net: A?.~ (VIN), M?.~ (VCC) (x3)
- now unconnected: Z?.~ (GND)
Other:
- note added: "Batteriies"
- note added: "Button unused"
- note added: "Resistor optional"
- note removed: "Battery"
- note removed: "Resistor is optional"
- note removed: "Switch is unused"
- moved on the sheet: A?, M?, R?, SW?, Z?
